Commit message: ajout du sol et ajustement security

File: src/universal_robot/ur_description/urdf/inc/ur_macro.xacro (robot description, xacro)
@@ -377,7 +377,7 @@
     <link name="${prefix}fake_gripper">
       <collision>
-        <origin xyz="0 0 0.12" rpy="0 0 0"/>
-        <geometry>
-          <box size="0.08 0.02 0.04"/>
+        <origin xyz="0 0 0.07" rpy="0 0 0"/>
+        <geometry>
+          <box size="0.08 0.08 0.30"/>
         </geometry>
       </collision>
